Commit message: fix links in urdf

File: robots/kinova/urdf/jaco.urdf (robot description, URDF)
Before this commit: robot jaco, 17 links, 16 joints
Links:
- link j2s7s300_link_1: geometry collision mesh filename=package://kinova/meshes/shoulder.dae; visual mesh filename=package://kinova/meshes/ring_big.STL
- link j2s7s300_link_2: geometry collision mesh filename=package://kinova/meshes/arm_half_1.dae; visual mesh filename=package://kinova/meshes/arm_half_1.dae
- link j2s7s300_link_3: geometry collision mesh filename=package://kinova/meshes/arm_half_2.dae; visual mesh filename=package://kinova/meshes/arm_half_2.dae
- link j2s7s300_link_4: geometry collision mesh filename=package://kinova/meshes/forearm.dae; visual mesh filename=package://kinova/meshes/forearm.dae
- link j2s7s300_link_5: geometry collision mesh filename=package://kinova/meshes/wrist_spherical_1.dae; visual mesh filename=package://kinova/meshes/ring_small.STL
- link j2s7s300_link_6: geometry collision mesh filename=package://kinova/meshes/wrist_spherical_2.dae; visual mesh filename=package://kinova/meshes/ring_small.STL
- link j2s7s300_link_7: geometry collision mesh filename=package://kinova/meshes/hand_3finger.dae; visual mesh filename=package://kinova/meshes/hand_3finger.dae
- link j2s7s300_link_base: geometry collision mesh filename=package://kinova/meshes/base.dae; visual mesh filename=package://kinova/meshes/base.dae
- link j2s7s300_link_finger_1: geometry collision mesh filename=package://kinova/meshes/finger_proximal.dae; visual mesh filename=package://kinova/meshes/finger_proximal.dae
- link j2s7s300_link_finger_2: geometry collision mesh filename=package://kinova/meshes/finger_proximal.dae; visual mesh filename=package://kinova/meshes/finger_proximal.dae
- link j2s7s300_link_finger_3: geometry collision mesh filename=package://kinova/meshes/finger_proximal.dae; visual mesh filename=package://kinova/meshes/finger_proximal.dae
- link j2s7s300_link_finger_tip_1: geometry collision mesh filename=package://kinova/meshes/finger_distal.dae; visual mesh filename=package://kinova/meshes/finger_distal.dae
- link j2s7s300_link_finger_tip_2: geometry collision mesh filename=package://kinova/meshes/finger_distal.dae; visual mesh filename=package://kinova/meshes/finger_distal.dae
- link j2s7s300_link_finger_tip_3: geometry collision mesh filename=package://kinova/meshes/finger_distal.dae; visual mesh filename=package://kinova/meshes/finger_distal.dae

File: robots/kinova/urdf/mico.urdf (robot description, URDF)
Before this commit: robot m1n6s200, 14 links, 13 joints
Links:
- link m1n6s200_link_1: geometry collision mesh filename=package://kinova/meshes/shoulder.dae; visual mesh filename=package://kinova/meshes/ring_big.STL
- link m1n6s200_link_2: geometry collision mesh filename=package://kinova/meshes/arm_mico.dae; visual mesh filename=package://kinova/meshes/arm_mico.dae
- link m1n6s200_link_3: geometry collision mesh filename=package://kinova/meshes/forearm_mico.dae; visual mesh filename=package://kinova/meshes/forearm_mico.dae
- link m1n6s200_link_4: geometry collision mesh filename=package://kinova/meshes/wrist.dae; visual mesh filename=package://kinova/meshes/ring_small.STL
- link m1n6s200_link_5: geometry collision mesh filename=package://kinova/meshes/wrist.dae; visual mesh filename=package://kinova/meshes/ring_small.STL
- link m1n6s200_link_6: geometry collision mesh filename=package://kinova/meshes/hand_2finger.dae; visual mesh filename=package://kinova/meshes/hand_2finger.dae
- link m1n6s200_link_base: geometry collision mesh filename=package://kinova/meshes/base.dae; visual mesh filename=package://kinova/meshes/base.dae
- link m1n6s200_link_finger_1: geometry collision mesh filename=package://kinova/meshes/finger_proximal.dae; visual mesh filename=package://kinova/meshes/finger_proximal.dae
- link m1n6s200_link_finger_2: geometry collision mesh filename=package://kinova/meshes/finger_proximal.dae; visual mesh filename=package://kinova/meshes/finger_proximal.dae
- link m1n6s200_link_finger_tip_1: geometry collision mesh filename=package://kinova/meshes/finger_distal.dae; visual mesh filename=package://kinova/meshes/finger_distal.dae
- link m1n6s200_link_finger_tip_2: geometry collision mesh filename=package://kinova/meshes/finger_distal.dae; visual mesh filename=package://kinova/meshes/finger_distal.dae
