Commit message: new meshes for spot arm

File: robots/spot_arm/urdf/spot_arm.urdf (robot description, URDF)
Before this commit: robot spot_arm, 28 links, 27 joints
Links:
- removed link finger_tip
- link base_arm_link: geometry collision mesh filename=package://spot_arm/meshes/arm/spot_0.dae; visual mesh filename=package://spot_arm/meshes/arm/spot_0.dae
- link finger: geometry collision mesh filename=package://spot_arm/meshes/arm/spot_7.dae; visual mesh filename=package://spot_arm/meshes/arm/spot_7.dae
- link gripper: geometry collision mesh filename=package://spot_arm/meshes/arm/spot_6.dae; visual mesh filename=package://spot_arm/meshes/arm/spot_6.dae
- link link1: geometry collision mesh filename=package://spot_arm/meshes/arm/spot_1.dae; visual mesh filename=package://spot_arm/meshes/arm/spot_1.dae
- link link2: geometry collision mesh filename=package://spot_arm/meshes/arm/spot_2.dae; visual mesh filename=package://spot_arm/meshes/arm/spot_2.dae
- link link3: geometry collision mesh filename=package://spot_arm/meshes/arm/spot_3.dae; visual mesh filename=package://spot_arm/meshes/arm/spot_3.dae
- link link4: geometry collision mesh filename=package://spot_arm/meshes/arm/spot_4.dae; visual mesh filename=package://spot_arm/meshes/arm/spot_4.dae
- link wrist: geometry collision mesh filename=package://spot_arm/meshes/arm/spot_5.dae; visual mesh filename=package://spot_arm/meshes/arm/spot_5.dae
Joints:
- removed joint finger_tip_joint
- joint arm_gripper: origin xyz=-0.86859 0.043915 -0.029 rpy=0 0 0 -> xyz=0.078 0 0.025 rpy=0 0 0
- joint arm_joint1: origin xyz=0.0 0.0 0.065 rpy=0 0 1.5707963267948966 -> xyz=0.0 0.0 0.065 rpy=0 0 0
- joint arm_joint2: axis 1.0 0.0 0.0 -> 0.0 1.0 0.0; origin xyz=0.015 0.0 0.05 rpy=-3.141592653589793 0 0 -> xyz=0.0 0.0 0.05 rpy=0 0 0
- joint arm_joint3: axis 1.0 0.0 0.0 -> 0.0 1.0 0.0; origin xyz=0.002 0.3125 0.0 rpy=0 0 0 -> xyz=0.3125 0.00 0.0 rpy=0 0 0
- joint arm_joint4: axis 0.0 1.0 0.0 -> 1.0 0.0 0.0; origin xyz=-0.018 0.138 -0.0675 rpy=0 0 0 -> xyz=0.138 0.0 0.075 rpy=0 0 0
- joint arm_joint5: axis 1.0 0.0 0.0 -> 0.0 1.0 0.0; origin xyz=-0.0475 0.24809 0.0 rpy=0 0 0 -> xyz=0.283 0 0.0 rpy=0 0 0
- joint arm_joint6: axis -0.0 1.0 0.0 -> 1.0 0.0 0.0; origin xyz=0.04 0.081 0.0 rpy=0 0 0 -> xyz=0.056 0.0 0.0 rpy=0 0 0
- joint base_link_joint: child base_link -> body; origin xyz=0 0 0 rpy=0 0 0 -> xyz=0 0 0.4 rpy=0 0 0; parent body -> base_link
- joint tool_tip_joint: origin xyz=0.0 0.2 0.0 rpy=-1.570796 0 0 -> xyz=0.2 0.0 0.0 rpy=0 1.570796 0
